File: hardware/board/microgame.kicad_pcb (KiCad board)
At the start: 2 copper layers, 25.5 x 33.7 mm, 25 parts, among them U1 ATTINY85-20SU

Commit message: Moved the button to the back.
Parts:
- S1: moved to B.Cu
- moved S1 16.0 mm to (141.0, 87.5), turned to 0 degrees
- moved C1 2.95 mm to (146.0, 99.0)
- moved U1 2.50 mm to (141.0, 100.0)
- turned BAT1 to 180 degrees
Routing:
- net LED4: track 68.4 -> 0.00 mm, vias 4 -> 0
- net LED2: track 58.8 -> 0.00 mm
- net LED3: track 51.3 -> 0.00 mm, vias 2 -> 0
- net LED5: track 49.8 -> 0.00 mm, vias 2 -> 0
- net LED1: track 49.2 -> 0.00 mm, vias 2 -> 0
- net GND: track 41.4 -> 0.00 mm, vias 2 -> 0
- net VCC: track 41.2 -> 0.00 mm, vias 1 -> 0
- net Net-(D10-Pad1): track 17.4 -> 0.00 mm
- net Net-(D13-Pad1): track 14.1 -> 0.00 mm
- net Net-(D1-Pad1): track 14.0 -> 0.00 mm
- net Net-(D5-Pad1): track 13.0 -> 0.00 mm
- net BUTTON: track 6.86 -> 0.00 mm

Commit message: Updated design to have a sane pin mapping. Added initial simulator program and firmware.
Connections:
- D1 pad 2: LED4 -> LED2
- D10 pad 2: LED3 -> LED2
- D11 pad 2: LED5 -> LED4
- D12 pad 2: LED1 -> LED5
- D13 pad 2: LED4 -> LED1
- D14 pad 2: LED5 -> LED2
- D15 pad 2: LED2 -> LED3
- D16 pad 2: LED1 -> LED5
- D3 pad 2: LED2 -> LED4
- D4 pad 2: LED1 -> LED5
- D5 pad 2: LED4 -> LED1
- D7 pad 2: LED2 -> LED4
- D9 pad 2: LED4 -> LED1
- R1 pad 2: LED5 -> LED1
- R2 pad 2: LED1 -> LED2
- R3 pad 2: LED2 -> LED3
- R4 pad 2: LED3 -> LED4
Routing:
- net LED5: track 0.00 -> 68.8 mm, vias 0 -> 4
- net LED1: track 0.00 -> 64.9 mm, vias 0 -> 3
- net LED2: track 0.00 -> 57.1 mm
- net LED4: track 0.00 -> 56.6 mm
- net LED3: track 0.00 -> 51.4 mm, vias 0 -> 2
- net VCC: track 0.00 -> 45.6 mm, vias 0 -> 1
- net GND: track 0.00 -> 44.4 mm, vias 0 -> 2
- net BUTTON: track 0.00 -> 19.2 mm, vias 0 -> 1
- net Net-(D1-Pad1): track 0.00 -> 14.1 mm
- net Net-(D13-Pad1): track 0.00 -> 13.8 mm
- net Net-(D5-Pad1): track 0.00 -> 13.0 mm
- net Net-(D10-Pad1): track 0.00 -> 12.9 mm
Other:
- board text added: "Press me!"
- board text added: "V1"

Commit message: Updated BOM
Parts:
- BAT1: value BS-7 -> Keystone 3034
- U1: value ATTINY85-20SU -> ATTINY25-20SSU
Changed lines of the file:
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@@
 			)
 		)
-		(property "Value" "ATTINY85-20SU"
+		(property "Value" "ATTINY25-20SSU"
 			(at 0 4.25 0)
 			(layer "F.Fab")
@@
 			)
 		)
-		(property "Value" "BS-7"
+		(property "Value" "Keystone 3034"
 			(at 0 -7.842529 0)
 			(layer "B.Fab")
